Commit message: two axis

File: src/two_axis_description/urdf/two_axis.urdf (robot description, URDF)
Before this commit: robot Two axis URDF, 3 links, 2 joints
Links:
- removed link Last_link
- removed link Middle_link
- added link Link_1, mass 0.12498; collision mesh filename=package://two_axis_description/meshes/link_1.STL scale=0.01 0.01 0.01; visual mesh filename=package://two_axis_description/meshes/link_1.STL scale=0.01 0.01 0.01
- added link Link_2, mass 0.13201; collision mesh filename=package://two_axis_description/meshes/link_2.STL; visual mesh filename=package://two_axis_description/meshes/link_2.STL scale=0.01 0.01 0.01
- added link world
- link base_link: mass 0.98158 -> 1.0009; geometry collision mesh filename=package://two_axis_description/meshes/base_link.STL; visual mesh filename=package://two_axis_description/meshes/base_link.STL scale=0.01 0.01 0.01
Joints:
- added joint world2base: type fixed, parent world, child base_link, origin xyz=0.0 0.0 0.0 rpy=0.0 0.0 0.0, axis 0.0 0.0 0.0, limit lower=0.0 upper=0.0 effort=0.0 velocity=0.0
- joint Joint_1: axis 0 0 -1 -> 0 1 0; child Middle_link -> Link_1; origin xyz=0 0 0 rpy=0 0 0 -> xyz=0 0 1.32 rpy=0 0 0
- joint Joint_2: axis -0.99989 -0.015041 0 -> 1 0 0; child Last_link -> Link_2; origin xyz=0 0 0 rpy=0 0 0 -> xyz=0.020 1.05 -0.6 rpy=0 -1.575 0; parent Middle_link -> Link_1

Commit message: fix collisions

File: src/two_axis_description/urdf/two_axis.urdf (robot description, URDF)
Before this commit: robot two_axis, 4 links, 3 joints
Links:
- removed link world
- link Link_2: geometry collision mesh filename=package://two_axis_description/meshes/link_2.STL scale=0.01 0.01 0.01; visual mesh filename=package://two_axis_description/meshes/link_2.STL scale=0.01 0.01 0.01
- link base_link: geometry collision mesh filename=package://two_axis_description/meshes/base_link.STL scale=0.01 0.01 0.01; visual mesh filename=package://two_axis_description/meshes/base_link.STL scale=0.01 0.01 0.01
Joints:
- removed joint world2base

Commit message: fix mass

File: src/two_axis_description/urdf/two_axis.urdf (robot description, URDF)
Before this commit: robot two_axis, 3 links, 2 joints
Links:
- link Link_2: mass 0.13201 -> 0.013201
- link base_link: mass 1.0009 -> 100.0009
Joints:
- joint Joint_1: origin xyz=0 0 1.32 rpy=0 0 0 -> xyz=0 0 2.32 rpy=0 0 0
