Commit message: gimbal 2 axis

File: src/tutorial_description/urdf/gazebo.xacro (robot description, xacro)
@@ -1,4 +1,4 @@
 <robot xmlns:xacro="http://www.ros.org/wiki/xacro">
-    <gazebo>
+    <!-- <gazebo>
         <plugin filename="gz_ros2_control-system" name="gz_ros2_control::GazeboSimROS2ControlPlugin">
             <parameters>
@@ -6,5 +6,5 @@
             </parameters>
         </plugin>
-    </gazebo>
+    </gazebo> -->
     <gazebo reference="first_link">
         <mu1>0.2</mu1>
@@ -26,3 +26,25 @@
         </sensor>
     </gazebo>
+    <gazebo reference="imu_link">
+        <sensor name="camera" type="camera">
+            <pose> 0 0 0 0 0 0 </pose>
+            <visualize>true</visualize>
+            <update_rate>10</update_rate>
+            <camera>
+                <camera_info_topic>camera/camera_info</camera_info_topic>
+                <horizontal_fov>1.089</horizontal_fov>
+                <image>
+                    <format>R8G8B8</format>
+                    <width>640</width>
+                    <height>480</height>
+                </image>
+                <clip>
+                    <near>0.05</near>
+                    <far>8.0</far>
+                </clip>
+            </camera>
+            <topic>camera/image_raw</topic>
+            <!-- <gz_frame_id>camera_link_optical</gz_frame_id> -->
+        </sensor>
+    </gazebo>
 </robot>

File: src/tutorial_description/urdf/robot.xacro (robot description, xacro)
@@ -2,4 +2,5 @@
     <xacro:include filename="parameters.xacro" />
     <xacro:include filename="gazebo.xacro" />
+    <xacro:include filename="effort_control.xacro" />
     <link name="world" />
     <joint name="fixed_joint" type="fixed">
@@ -76,17 +77,9 @@
     <!-- #################################################### -->
     <!-- control plugin and definition -->
-    <ros2_control name="robot" type="system">
+    <!-- <ros2_control name="robot" type="system">
         <hardware>
             <plugin>gz_ros2_control/GazeboSimSystem</plugin>
         </hardware>
         <joint name="first_joint">
-            <!-- <command_interface name="position">
-                <param name="min">-1.571</param>
-                <param name="max">1.571</param>
-            </command_interface> -->
-            <!-- <command_interface name="velocity">
-                <param name="min">-2.0</param>
-                <param name="max">2.0</param>
-            </command_interface> -->
             <command_interface name="effort">
                 <param name="min">-2.0</param>
@@ -106,7 +99,6 @@
             <state_interface name="linear_acceleration.y" />
             <state_interface name="linear_acceleration.z" />
-            <!-- <param name="frame_id">second_link</param> -->
         </sensor>
-    </ros2_control>
+    </ros2_control> -->
     <!-- #################################################### -->
 </robot>

File: src/two_axis_description/urdf/two_axis.urdf (robot description, URDF)
Before this commit: robot two_axis, 3 links, 2 joints
Joints:
- joint Joint_1: limit lower=-1.57 upper=1.57 effort=0.147 velocity=87 -> lower=-1.57 upper=1.57 effort=100 velocity=87
- joint Joint_2: limit lower=-1.57 upper=1.57 effort=0.147 velocity=87 -> lower=-1.57 upper=1.57 effort=100 velocity=87
